File: SwirlsV1.2/SwirlsV1.2.sch (EAGLE design)
At the start: 130 parts, among them IC1 LM1117-3.3, IC2 LM4040B25, IC3 LM1117-3.3, IC4 DAC8552, IC5 TL072, IC6 TL072, IC7 LM4040B10, IC8 MCP6002, IC9 MCP6004, J1 PJ301_GUI6, J10 PJ301_GUI6, J11 PJ301_GUI6, J12 PJ301_GUI6, J13 PJ301_GUI6, J2 PJ301_GUI6, J3 PJ301_GUI6, J4 PJ301_GUI6, J5 PJ301_GUI6, J6 PJ301_GUI6, J7 PJ301_GUI6, J8 PJ301_GUI6, J9 PJ301_GUI6, Q1 8MHz, Q2 MMBT3904, Q3 MMBT3904, Q4 MMBT3904, Q5 MMBT3904, Q6 MMBT3904, SW3 TL1100X, SW4 TL1100X

Commit message: fixed
Parts:
- removed D1, D2: 1N5819HW, diode:DIODE-SOD123
- removed POWER: M05X2PTH, og-header:M05X2PTH
- removed Q1: 8MHz, SparkFun-Clocks:CRYSTAL-8MHZSMD-HC49UP
- added G1: (no value), microbuilder:BRIDGERECTIFIER
- added JP2: M05X2PTH, braids_v50:M05X2PTH
- added X1: (no value), Icotech_Eagle_Library:XTALNX5032
- C10, C3: device rcl:CPOL-USD -> rcl:CPOL-USC
- R6: value 10k -> 10kb
Connections:
- removed net N$56: D1.A, POWER.1, POWER.2
- removed net N$64: D2.C, POWER.10, POWER.9
- new net N$49: G1.AC1, JP2.1, JP2.2
- new net N$50: G1.AC2, JP2.10, JP2.9
- net GND: now also JP2.3, JP2.4, JP2.5, JP2.6, JP2.7, JP2.8; no longer POWER.3, POWER.4, POWER.5, POWER.6, POWER.7, POWER.8
- net N$7: now also X1.P$2; no longer Q1.2
- net N$8: now also X1.P$1; no longer Q1.1
- net VCC: now also G1.+; no longer D1.C
- net VEE: now also G1.-; no longer D2.A
